File: pcb/ardwiino.kicad_pcb (KiCad board)
At the start: 2 copper layers, 64 x 26.4 mm, 9 parts, among them M1 Top, U1 ProMicro

Commit message: remove mounting holes
Parts:
- removed REF** (x4): MountingHole_3.2mm_M3_DIN965, MountingHole:MountingHole_3.2mm_M3_DIN965
Changed lines of the file:
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@@
-(kicad_pcb (version 20171130) (host pcbnew "(5.0.1)-3")
+(kicad_pcb (version 20171130) (host pcbnew "(5.0.1-3-g963ef8bb5)")
   (general
     (thickness 1.6)
@@
     (tracks 51)
     (zones 0)
-    (modules 9)
+    (modules 5)
     (nets 28)
   )
@@
     (add_net "Net-(MPU6050-Pad8)")
   )
-  (module MountingHole:MountingHole_3.2mm_M3_DIN965 (layer F.Cu)
-    (at 123.825 68.58)
-    (descr "Mounting Hole 3.2mm, no annular, M3, DIN965")
-    (tags "mounting hole 3.2mm no annular m3 din965")
-    (attr virtual)
-    (fp_text reference REF** (at 0 -3.8) (layer F.SilkS) hide
-      (effects (font (size 1 1) (thickness 0.15)))
-    )
-    (fp_text value MountingHole_3.2mm_M3_DIN965 (at 0 -6.604) (layer F.Fab) hide
-      (effects (font (size 1 1) (thickness 0.15)))
-    )
-    (fp_text user %R (at 0.3 0) (layer F.Fab)
-      (effects (font (size 1 1) (thickness 0.15)))
-    )
-    (fp_circle (center 0 0) (end 2.8 0) (layer Cmts.User) (width 0.15))
-    (fp_circle (center 0 0) (end 3.05 0) (layer F.CrtYd) (width 0.05))
-    (pad 1 np_thru_hole circle (at 0 0) (size 3.2 3.2) (drill 3.2) (layers *.Cu *.Mask))
-  )
-  (module MountingHole:MountingHole_3.2mm_M3_DIN965 (layer F.Cu)
-    (at 123.825 88.9)
-    (descr "Mounting Hole 3.2mm, no annular, M3, DIN965")
-    (tags "mounting hole 3.2mm no annular m3 din965")
-    (attr virtual)
-    (fp_text reference REF** (at 0 -3.8) (layer F.SilkS)
-      (effects (font (size 1 1) (thickness 0.15)))
-    )
-    (fp_text value MountingHole_3.2mm_M3_DIN965 (at 0 -6.604) (layer F.Fab) hide
-      (effects (font (size 1 1) (thickness 0.15)))
-    )
-    (fp_text user %R (at 0.3 0) (layer F.Fab)
-      (effects (font (size 1 1) (thickness 0.15)))
-    )
-    (fp_circle (center 0 0) (end 2.8 0) (layer Cmts.User) (width 0.15))
-    (fp_circle (center 0 0) (end 3.05 0) (layer F.CrtYd) (width 0.05))
-    (pad 1 np_thru_hole circle (at 0 0) (size 3.2 3.2) (drill 3.2) (layers *.Cu *.Mask))
-  )
-  (module MountingHole:MountingHole_3.2mm_M3_DIN965 (layer F.Cu)
-    (at 148.463 88.9)
-    (descr "Mounting Hole 3.2mm, no annular, M3, DIN965")
-    (tags "mounting hole 3.2mm no annular m3 din965")
-    (attr virtual)
-    (fp_text reference REF** (at 0 -3.8) (layer F.SilkS) hide
-      (effects (font (size 1 1) (thickness 0.15)))
-    )
-    (fp_text value MountingHole_3.2mm_M3_DIN965 (at 0 -6.604) (layer F.Fab) hide
-      (effects (font (size 1 1) (thickness 0.15)))
-    )
-    (fp_text user %R (at 0.3 0) (layer F.Fab)
-      (effects (font (size 1 1) (thickness 0.15)))
-    )
-    (fp_circle (center 0 0) (end 2.8 0) (layer Cmts.User) (width 0.15))
-    (fp_circle (center 0 0) (end 3.05 0) (layer F.CrtYd) (width 0.05))
-    (pad 1 np_thru_hole circle (at 0 0) (size 3.2 3.2) (drill 3.2) (layers *.Cu *.Mask))
-  )
   (module ProMicro:ProMicro (layer F.Cu)
     (at 105.41 78.74)
@@
     )
   )
-  (module MountingHole:MountingHole_3.2mm_M3_DIN965 (layer F.Cu)
-    (at 148.463 68.58)
-    (descr "Mounting Hole 3.2mm, no annular, M3, DIN965")
-    (tags "mounting hole 3.2mm no annular m3 din965")
-    (attr virtual)
-    (fp_text reference REF** (at 0 -3.8) (layer F.SilkS) hide
-      (effects (font (size 1 1) (thickness 0.15)))
-    )
-    (fp_text value MountingHole_3.2mm_M3_DIN965 (at 0 -6.604) (layer F.Fab) hide
-      (effects (font (size 1 1) (thickness 0.15)))
-    )
-    (fp_circle (center 0 0) (end 3.05 0) (layer F.CrtYd) (width 0.05))
-    (fp_circle (center 0 0) (end 2.8 0) (layer Cmts.User) (width 0.15))
-    (fp_text user %R (at 0.3 0) (layer F.Fab)
-      (effects (font (size 1 1) (thickness 0.15)))
-    )
-    (pad 1 np_thru_hole circle (at 0 0) (size 3.2 3.2) (drill 3.2) (layers *.Cu *.Mask))
-  )
   (gr_text "Ardwiino V1.0\nSanjay Govind\nSebastiaan Jansen" (at 131.699 79.375) (layer B.SilkS)
